File: RPi Hat RF Transmitter V1.kicad_pcb (KiCad board)
At the start: 4 copper layers, 65 x 56 mm, 83 parts, among them CON1 Sig_In, CON2 SMA-, IC1 ADG904BRUZ-R, IC3 SN74HC139PW, IC4 ADG904BRUZ-R, J1 Conn_02x03_Odd_Even, J10 U.FL-R-SMT(10), J11 U.FL-R-SMT(10), J12 U.FL-R-SMT(10), J3 40HAT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

Commit message: before generating GERBER
Routing:
- net GND: vias 111 -> 113

Commit message: adds silk screen updates, ground stiching and generated GERBERs
Parts:
- added TP1: TestPoint, Connector_Pin:Pin_D0.9mm_L10.0mm_W2.4mm_FlatFork, F.Cu at (108.2, 102.2)
Routing:
- net RF_SWITCH_PWR: track 119.4 -> 130.8 mm, vias 6 -> 7
- net GND: vias 113 -> 375
Other:
- board text added: "2.5V SUPPLY EN"
- board text added: "A0"
- board text added: "A1"
- board text added: "ADG904"
- board text added: "IC1, IC4"
- board text added: "JP5"
- board text added: "JP6"
- board text added: "RF IN FROM RPI"
- board text added: "RF S EN"
- board text added: "U3"
- board text removed: "A"
- board text removed: "B"
- board text removed: "HMC241"
- board text removed: "IC1, IC2"
- board text removed: "U2"
