File: RPi Hat RF Transmitter V1.sch (KiCad schematic (older format))
At the start: 67 parts, among them CON1 Sig_In, CON2 SMA-, CON3 Sig_In, CON4 Sig_In, CON5 SMA-, IC1 HMC241AQS16E, IC2 HMC241AQS16E, IC3 SN74HC139PW, J1 Conn_01x04_Male, J2 Conn_01x04_Male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

Commit message: changes the switch, adds LDO, adds Jumpers for RF lines, changes names of existing nets
Parts:
- removed IC1, IC2: HMC241AQS16E, SamacSys_Parts:SOP64P600X175-16N, symbol SamacSys_Parts:HMC241AQS16E
- removed J1: Conn_01x04_Male, Connector_PinHeader_2.54mm:PinHeader_1x04_P2.54mm_Vertical, symbol Connector:Conn_01x04_Male
- removed R15: 330, Resistor_SMD:R_0805_2012Metric_Pad1.15x1.40mm_HandSolder, symbol Device:R
- removed U2: 74AUC2G04, Package_TO_SOT_SMD:SOT-23-6_Handsoldering, symbol 74xGxx:74AUC2G04
- added C? (x2): 0.1uF, Capacitor_SMD:C_0805_2012Metric_Pad1.15x1.40mm_HandSolder, symbol Device:C
- added C? (x2): 10uF, Capacitor_SMD:C_0805_2012Metric_Pad1.15x1.40mm_HandSolder, symbol Device:C
- added C?: 10uF, Capacitor_SMD:C_1206_3216Metric_Pad1.42x1.75mm_HandSolder, symbol Device:C
- added C? (x2): 22uF, Capacitor_SMD:C_1206_3216Metric_Pad1.42x1.75mm_HandSolder, symbol Device:C
- added IC? (x2): ADG904BRUZ-R, SOP65P640X120-20N, symbol SamacSys_Parts:ADG904BRUZ-R
- added IC?: SN74HC139PW, Package_SO:TSSOP-16_4.4x5mm_P0.65mm, symbol SamacSys_Parts:SN74HC139PW
- added J? (x2): Conn_01x03_Male, Connector_PinHeader_2.54mm:PinHeader_1x03_P2.54mm_Vertical, symbol Connector:Conn_01x03_Male
- added J?: Conn_01x08_Male, symbol Connector:Conn_01x08_Male
- added JP? (x4): Jumper, Connector_PinHeader_2.54mm:PinHeader_1x02_P2.54mm_Vertical, symbol Device:Jumper
- added R? (x4): 330, Resistor_SMD:R_0805_2012Metric_Pad1.15x1.40mm_HandSolder, symbol Device:R
- added R? (x2): 10K, Resistor_SMD:R_0805_2012Metric_Pad1.15x1.40mm_HandSolder, symbol Device:R
- added R? (x2): 120, Resistor_SMD:R_0805_2012Metric_Pad1.15x1.40mm_HandSolder, symbol Device:R
- added U?: LM1117-ADJ, Package_TO_SOT_SMD:SOT-223-3_TabPin2, symbol Regulator_Linear:AZ1117-ADJ
Connections:
- net labels added: A0_1, A0_2, A1_1, A1_2, DECODER_EN, FIL_IN_1, FIL_IN_2, FIL_IN_3, FIL_IN_4, FIL_OUT_1, FIL_OUT_2, FIL_OUT_3, FIL_OUT_4, RF_SWITCH_EN, RF_SWITCH_IN, RF_SWITCH_OUT, RPI_RF_OUT
- net labels removed: GPIO17, GPIO22, GPIO27, GPIO4, P5V, P5V_HAT, RF1_IN, RF1_OUT, RF2_IN, RF2_OUT, RF3_IN, RF3_OUT, RF4_IN, RF4_OUT, RF_ANT_OUT, RF_IN_SWITCH
- wire segments 271 -> 329
- no-connect marks 36 -> 40
Other:
- note removed: "5V Powered HAT Protection"
- note removed: "This is based on the official Raspberry Pi spec to be able to call an extension board a HAT.\nhttps://github.com/raspberrypi/hats/blob/master/designguide.md"
- note removed: "This is the recommended 5V rail protection for \na HAT with power going to the Pi.\nSee https://github.com/raspberrypi/hats/blob/master/designguide.md#back-powering-the-pi-via-the-j8-gpio-header"
- moved on the sheet: C13, C14, C15, C16, C17, CON1, CON2, CON5, D5, D6, D7, J2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

Commit message: adds ufl connectors, now readymade filter at forth filter etc
Parts:
- removed CON3, CON4: Sig_In, Connector_Coaxial:SMA_Amphenol_132291-12_Vertical, symbol vk_custom_kicad:SMA-
- removed CON5: SMA-, Connector_Coaxial:SMA_Amphenol_132291-12_Vertical, symbol vk_custom_kicad:SMA-
- removed JP? (x2): Jumper, Connector_PinHeader_2.54mm:PinHeader_1x02_P2.54mm_Vertical, symbol Device:Jumper
- removed R12, R13, R14: 330, Resistor_SMD:R_0805_2012Metric_Pad1.15x1.40mm_HandSolder, symbol Device:R
- added FIL4: LFCN-180, Filter:Filter_Mini-Circuits_FV1206, symbol RF_Filter:LFCN-180
- added J10, J11, J12, J9: U.FL-R-SMT(10), SamacSys_Parts:UFLRSMT10, symbol SamacSys_Parts:U.FL-R-SMT(10)
- added R1: 330, Resistor_SMD:R_0805_2012Metric_Pad1.15x1.40mm_HandSolder, symbol Device:R
- IC1, IC4: renamed from IC?; footprint SOP65P640X120-20N -> SamacSys_Parts:SOP65P640X120-20N
- J1: renamed from J?; footprint (none) -> Connector_PinHeader_2.54mm:PinHeader_1x08_P2.54mm_Vertical
- gave numbers to parts that had none: 21
Connections:
- net +5V: now also J2.3 (Pin_3), J2.4 (Pin_4); no longer J2.1 (Pin_1), J2.2 (Pin_2), J5.1 (Pin_1), J6.1 (Pin_1), J7.1 (Pin_1), J8.1 (Pin_1), R5.2
- net A0_1: no longer J5.2 (Pin_2)
- net A0_2: no longer J6.2 (Pin_2)
- net A1_1: no longer J7.2 (Pin_2)
- net A1_2: no longer J8.2 (Pin_2)
- net FIL_IN_4: now also FIL4.1 (IN), J9.3 (SIG)
- net FIL_OUT_4: now also FIL4.3 (OUT), J10.3 (SIG)
- net GND: now also J2.1 (Pin_1), J2.2 (Pin_2), FIL4.2 (GND), FIL4.4 (GND), J10.1 (GND_1), J10.2 (GND_2), J11.1 (GND_1), J11.2 (GND_2), J12.1 (GND_1), J12.2 (GND_2), J9.1 (GND_1), J9.2 (GND_2); no longer J2.3 (Pin_3), J2.4 (Pin_4)
- net RF_SWITCH_EN: now also R1.2; no longer IC1.1 (~EN), IC4.1 (~EN), R2.2
- net at C13.1: now also J11.3 (SIG)
- net A1_1_JMP: now reaches IC1.19 (A1), R4.2
- net A1_1_JMP: now also J7.2 (Pin_2)
- net A0_1_JMP: now reaches IC1.20 (A0), R3.2
- net A0_1_JMP: now also J5.2 (Pin_2)
- net DECODER_PWR: now reaches C6.1, JP2.2, U2.3 (VI)
- net DECODER_PWR: now also C19.1, IC2.16 (VCC), IC3.16 (VCC), R5.2
- net A1_2_JMP: now reaches IC4.19 (A1), R15.2
- net A1_2_JMP: now also J8.2 (Pin_2)
- net A0_2_JMP: now reaches IC4.20 (A0), R9.2
- net A0_2_JMP: now also J6.2 (Pin_2)
- net at D1.1 (K), R11.2: now also D2.1 (K), D3.1 (K), D4.1 (K)
- net RF_SWITCH_IN: no longer names the net of CON1.1, IC1.10 (RFC), JP5.2
- net RF_SWITCH_OUT: no longer names the net of IC4.10 (RFC)
- net RF_SWITCH_OUT: now also J12.3 (SIG)
- net RF_SWITCH_PWR renamed +2V5
- net +2V5: now also J5.1 (Pin_1), J6.1 (Pin_1), J7.1 (Pin_1), J8.1 (Pin_1); no longer C19.1, IC2.16 (VCC), IC3.16 (VCC)
- new net: IC1.1 (~EN), IC4.1 (~EN), R1.1, R2.2
Other:
- moved on the sheet: C13, C14, C15, C16, C17, C2, C4, CON1, CON2, D1, D2, D3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

Commit message: routed for new circuit
Parts:
- removed IC2: SN74HC139PW, Package_SO:TSSOP-16_4.4x5mm_P0.65mm, symbol SamacSys_Parts:SN74HC139PW
- removed J1: Conn_01x08_Male, Connector_PinHeader_2.54mm:PinHeader_1x08_P2.54mm_Vertical, symbol Connector:Conn_01x08_Male
- removed J2: Conn_01x04_Male, Connector_PinHeader_2.54mm:PinHeader_1x04_P2.54mm_Vertical, symbol Connector:Conn_01x04_Male
- removed J6, J8: Conn_01x03_Male, Connector_PinHeader_2.54mm:PinHeader_1x03_P2.54mm_Vertical, symbol Connector:Conn_01x03_Male
- removed R15, R9: 330, Resistor_SMD:R_0805_2012Metric_Pad1.15x1.40mm_HandSolder, symbol Device:R
- added J1: Conn_02x03_Odd_Even, Connector_PinHeader_2.54mm:PinHeader_2x03_P2.54mm_Vertical, symbol Connector_Generic:Conn_02x03_Odd_Even
- added R12, R13: DNP, Resistor_SMD:R_0603_1608Metric, symbol Device:R
- added U3: 74AUC2G04, Package_TO_SOT_SMD:SOT-23-6_Handsoldering, symbol 74xGxx:74AUC2G04
Connections:
- net A1_2_JMP is gone; now on net A1_JMP: IC4.19 (A1)
- net +2V5: now also C19.1, IC3.16 (VCC), J5.3 (Pin_3), J7.3 (Pin_3), R11.2, R5.2, U3.5 (VCC); no longer J5.1 (Pin_1), J7.1 (Pin_1)
- net +5V: now also J1.2 (Pin_2)
- net GND: now also J5.1 (Pin_1), J7.1 (Pin_1), J1.1 (Pin_1), R13.1, U3.2 (GND); no longer D7.1 (K), J5.3 (Pin_3), J7.3 (Pin_3), JP3.1, R11.1
- net RF_SWITCH_EN: now also JP3.1, J1.5 (Pin_5)
- net SEL_RF1: now also D1.1 (K); no longer D1.2 (A)
- net SEL_RF2: now also D2.1 (K); no longer D2.2 (A)
- net SEL_RF3: now also D3.1 (K); no longer D3.2 (A)
- net SEL_RF4: now also D4.1 (K); no longer D4.2 (A)
- net RF_SWITCH_EN_STATUS: now reaches IC1.1 (~EN), IC4.1 (~EN), R1.1, R2.2
- net RF_SWITCH_EN_STATUS: now also R12.1
- net A0_1 renamed A0_RPI
- net A0_RPI: now also J1.4 (Pin_4); no longer IC3.2 (1A)
- net A0_1_JMP renamed A0_JMP
- net A0_JMP: now also IC3.2 (1A), U3.1
- net A0_2: no longer names the net of J3.17 (P3V3)
- net A0_2_JMP: no longer names the net of IC4.20 (A0)
- net A0_2_JMP: now also U3.6
- net A1_1 renamed A1_RPI
- net A1_RPI: now also J1.6 (Pin_6); no longer IC3.3 (1B)
- net A1_1_JMP renamed A1_JMP
- net A1_JMP: now also IC3.3 (1B)
- net A1_2: no longer names the net of J3.19 (BCM10)
- net DECODER_EN: no longer names the net of IC3.1 (~1G), JP3.2, R5.1
- net DECODER_EN: no longer J3.23 (BCM11)
- net DECODER_PWR: no longer names the net of C6.1, JP2.2, U2.3 (VI)
- net DECODER_PWR: no longer C19.1, IC3.16 (VCC), R5.2
- new net: D7.1 (K), R12.2, R13.2
- new net: D1.2 (A), D2.2 (A), D3.2 (A), D4.2 (A), R11.1
- no-connect marks 40 -> 37
Other:
- moved on the sheet: C10, C18, C19, C6, D1, D2, D3, D4, D5, D7, IC3, J4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

Commit message: adds silk screen updates, ground stiching and generated GERBERs
Parts:
- added TP1: TestPoint, Connector_Pin:Pin_D0.9mm_L10.0mm_W2.4mm_FlatFork, symbol Connector:TestPoint
Connections:
- net +2V5: now also TP1.1
Changed lines of the file:
@@
 Wire Wire Line
 	13375 2050 13550 2050
+$Comp
+L Connector:TestPoint TP1
+U 1 1 5DC2EB13
+P 13650 3850
+F 0 "TP1" H 13708 3968 50  0000 L CNN
+F 1 "TestPoint" H 13708 3877 50  0000 L CNN
+F 2 "Connector_Pin:Pin_D0.9mm_L10.0mm_W2.4mm_FlatFork" H 13850 3850 50  0001 C CNN
+F 3 "~" H 13850 3850 50  0001 C CNN
+	1    13650 3850
+	1    0    0    -1
+$EndComp
+Connection ~ 13650 3850
 $EndSCHEMATC
